Commit message: Add teleop teach replay and vision control stack

File: src/rebotarm_bringup/description/urdf/reBot-DevArm_fixend.urdf (robot description, URDF)
Before this commit: robot reBot-DevArm_fixend, 8 links, 7 joints
Links:
- added link left_finger_link; collision mesh filename=package://rebotarm_bringup/description/meshes/left_finger.s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; visual mesh filename=package://rebotarm_bringup/description/meshes/left_finger.s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
- added link right_finger_link; collision mesh filename=package://rebotarm_bringup/description/meshes/right_finger.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; visual mesh filename=package://rebotarm_bringup/description/meshes/right_finger.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
- link end_link: geometry collision mesh filename=package://rebotarm_bringup/description/meshes/gripper_base.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; visual mesh filename=package://rebotarm_bringup/description/meshes/gripper_base.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
Joints:
- added joint left_finger_joint: type prismatic, parent end_link, child left_finger_link, origin xyz=0 0 0 rpy=0 0 0, axis 0 1 0, limit lower=0.0 upper=0.045 effort=1.0 velocity=0.2
- added joint right_finger_joint: type prismatic, parent end_link, child right_finger_link, origin xyz=0 0 0 rpy=0 0 0, axis 0 1 0, limit lower=-0.045 upper=0.0 effort=1.0 velocity=0.2

File: src/rebotarm_moveit_config/config/rebotarm.urdf (robot description, URDF)
Before this commit: robot reBot-DevArm_fixend, 8 links, 7 joints
Links:
- added link left_finger_link; collision mesh filename=package://rebotarm_bringup/description/meshes/left_finger.s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; visual mesh filename=package://rebotarm_bringup/description/meshes/left_finger.s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
- added link right_finger_link; collision mesh filename=package://rebotarm_bringup/description/meshes/right_finger.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; visual mesh filename=package://rebotarm_bringup/description/meshes/right_finger.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
- link end_link: geometry collision mesh filename=package://rebotarm_bringup/description/meshes/gripper_base.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; visual mesh filename=package://rebotarm_bringup/description/meshes/gripper_base.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
Joints:
- added joint left_finger_joint: type prismatic, parent end_link, child left_finger_link, origin xyz=0 0 0 rpy=0 0 0, axis 0 1 0, limit lower=0.0 upper=0.045 effort=1.0 velocity=0.2
- added joint right_finger_joint: type prismatic, parent end_link, child right_finger_link, origin xyz=0 0 0 rpy=0 0 0, axis 0 1 0, limit lower=-0.045 upper=0.0 effort=1.0 velocity=0.2
