Commit message: feat: drive MuJoCo motors with simulated motor control

File: src/rebotarm_bringup/description/urdf/reBot-DevArm_fixend.urdf (robot description, URDF)
Before this commit: robot reBot-DevArm_fixend, 10 links, 9 joints
Joints:
- joint joint4: limit lower=-1.87 upper=1.57 effort=7 velocity=200 -> lower=-1.87 upper=1.57 effort=12.5 velocity=200
- joint joint5: limit lower=-1.57 upper=1.57 effort=7 velocity=200 -> lower=-1.57 upper=1.57 effort=12.5 velocity=200
- joint joint6: limit lower=-3.14 upper=3.14 effort=7 velocity=200 -> lower=-3.14 upper=3.14 effort=12.5 velocity=200

File: src/rebotarm_moveit_config/config/rebotarm.urdf (robot description, URDF)
Before this commit: robot reBot-DevArm_fixend, 10 links, 9 joints
Joints:
- joint joint4: limit lower=-1.87 upper=1.57 effort=7 velocity=200 -> lower=-1.87 upper=1.57 effort=12.5 velocity=200
- joint joint5: limit lower=-1.57 upper=1.57 effort=7 velocity=200 -> lower=-1.57 upper=1.57 effort=12.5 velocity=200
- joint joint6: limit lower=-3.14 upper=3.14 effort=7 velocity=200 -> lower=-3.14 upper=3.14 effort=12.5 velocity=200

Commit message: feat: migrate hardware safety and organize project documentation

File: src/rebotarm_bringup/description/urdf/reBot-DevArm_fixend.urdf (robot description, URDF)
Before this commit: robot reBot-DevArm_fixend, 10 links, 9 joints
Joints:
- joint joint4: limit lower=-1.87 upper=1.57 effort=12.5 velocity=200 -> lower=-1.87 upper=1.57 effort=7 velocity=200
- joint joint5: limit lower=-1.57 upper=1.57 effort=12.5 velocity=200 -> lower=-1.57 upper=1.57 effort=7 velocity=200
- joint joint6: limit lower=-3.14 upper=3.14 effort=12.5 velocity=200 -> lower=-3.14 upper=3.14 effort=7 velocity=200

File: src/rebotarm_moveit_config/config/rebotarm.urdf (robot description, URDF)
Before this commit: robot reBot-DevArm_fixend, 10 links, 9 joints
Joints:
- joint joint4: limit lower=-1.87 upper=1.57 effort=12.5 velocity=200 -> lower=-1.87 upper=1.57 effort=7 velocity=200
- joint joint5: limit lower=-1.57 upper=1.57 effort=12.5 velocity=200 -> lower=-1.57 upper=1.57 effort=7 velocity=200
- joint joint6: limit lower=-3.14 upper=3.14 effort=12.5 velocity=200 -> lower=-3.14 upper=3.14 effort=7 velocity=200
